File: PCB/kicad/LibreServo-v4.0.0.kicad_sch (KiCad schematic)
At the start: 105 parts, among them M1 M1, M2 MOSFET_N+P, M3 MOSFET_N+P, M4 FAN3227/4, M5 FAN3227/4, U1 M0G3518QRHBRQ1, U10 AEAT-8800, U2 MPM3610, U3 AP2112, U4 ACS711, U5 ADM2587E, U6 ADM3055E, U7 OPTIGA_TRUST_M

Commit message: chore(kicad): baseline reformat + plan for ERC/DRC clean-up
KiCad's own alphabetical lib_symbols reordering from an earlier GUI
session (confirmed no data loss: 65 lib symbols / 198 component
instances identical before and after). Also gitignores the KiCad
auto-backup and kicad-skill analysis-cache directories, and adds the
implementation plan for bringing the v4 schematic/PCB to ERC/DRC-clean,
manufacture-ready state (TODO.md 5.0-5.3, 6.1-6.3).

Co-Authored-By: Claude Sonnet 5 <noreply@anthropic.com>
Parts:
- renumbered C43 to C46
Connections:
- net +5V_ISO_CANFD is gone; now on net +3V3: C31.1, C32.1, U6.2 (VCC)
- net CAN0_RX is gone; now on net +3V3: U1.17 (PA13/CAN0_RX), U6.4 (RXD)
- net CAN0_TX is gone; now on net +3V3: U1.16 (PA12/CAN0_TX), U6.6 (TXD)
- net CANFD_ISO_GND is gone; now on net +3V3: #U$26.1 (P$1), #U$27.1 (P$1), B5.2, C37.2, C38.2, C41.2, U6.10 (RS), U6.9 (GND2)
- net GND is gone; now on net +3V3: C1.1, C10.2, C11.2, C12.1, C13.1, C14.2, C15.2, C16.1, C17.1, C18.1, C19.1, C2.1, C20.2, C21.2, C22.-, C23.2, C24.2, C25.2, C26.2, C3.2, C31.2, C32.2, C33.2, C34.2, C39.2, C4.2, C40.2, C42.2, C43.2, C44.2, C45.2, C46.2, C5.2, C6.2, C7.2, C8.1, C9.2, M1.P$1 (G), M2.P$1 (S1_N), M3.P$1 (S1_N), M4.P$3 (GND), M4.P$9 (TP), M5.P$3 (GND), M5.P$9 (TP), NTC0.1, R11.2, R12.2, R20.2, R4.1, U$100.P$2 (GND), U$3.P$4, U$4.P$2, U$5.P$3, U$6.P$3, U$8.P$2, U$9.P$2, U1.25 (PA21/VREF-), U1.33 (PAD), U1.5 (VSS), U10.P$13, U10.P$20, U10.P$25, U2.P$12 (P$8_PGND), U2.P$13 (P$8_PGND), U2.P$14 (P$8_PGND), U3.2 (P$2), U4.P$10, U4.P$5, U4.P$7, U4.P$8, U4.P$9, U5.2 (GND1), U6.1 (GND1), U6.5 (SILENT), U6.7 (STBY), U7.1 (GND)
- net +3V3: now also C33.1
Other:
- moved on the sheet: B4, B5, B6, B7, C13, C14, C15, C25, C26, C27, C28, C29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

Commit message: fix(sch): annotate 9 orphaned EAGLE-import components (U1)
U\$1/U\$2 (SLOT/SERVO_SLOT) -> J1/J2, U\$3/U\$4 (FFC-5) -> J4/J3,
U\$5 (HEADER_4_1.27_0.3) -> J5, U\$6 (POTEN_SERVO) -> RV1,
U\$8/U\$9 (JST_PH-4_HOLEB, RS-485 daisy-chain in/out) -> J6/J7,
U\$100 (OSCILATOR) -> Y1. Matches the existing #-prefix CAN-FD IN/OUT
JST connector pair's convention (in/out gets sequential same-family
refs). Resolves the "schematic has annotation errors" netlist-export
warning (TODO.md 6.1).

Verified: 117 components before and after, 0 duplicate reference
designators, 0 remaining U\$-form references (analyze_schematic.py).
ERC violation count unchanged (64) confirming no wiring was disturbed.

Co-Authored-By: Claude Sonnet 5 <noreply@anthropic.com>
Parts:
- renumbered U$1 to J1, U$2 to J2, U$4 to J3, U$3 to J4, U$5 to J5, U$8 to J6, U$9 to J7, U$6 to RV1, U$100 to Y1
Changed lines of the file:
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@@
 		(on_board yes)
 		(dnp no)
-		(property "Reference" "U$4"
+		(property "Reference" "J3"
 			(at 381 190.5 0)
 			(effects
@@
 			(project ""
 				(path "/f57eb5ac-0a1b-4ac0-915c-20e575439506"
-					(reference "U$4")
+					(reference "J3")
 					(unit 1)
 				)
@@
 		(on_board yes)
 		(dnp no)
-		(property "Reference" "U$2"
+		(property "Reference" "J2"
 			(at 495.3 134.62 0)
 			(effects
@@
 			(project ""
 				(path "/f57eb5ac-0a1b-4ac0-915c-20e575439506"
-					(reference "U$2")
+					(reference "J2")
 					(unit 1)
 				)
@@
 		(on_board yes)
 		(dnp no)
-		(property "Reference" "U$6"
+		(property "Reference" "RV1"
 			(at 487.68 205.74 0)
 			(effects
@@
 			(project ""
 				(path "/f57eb5ac-0a1b-4ac0-915c-20e575439506"
-					(reference "U$6")
+					(reference "RV1")
 					(unit 1)
 				)
@@
 		(on_board yes)
 		(dnp no)
-		(property "Reference" "U$8"
+		(property "Reference" "J6"
 			(at 467.36 218.44 90)
 			(effects
@@
 			(project ""
 				(path "/f57eb5ac-0a1b-4ac0-915c-20e575439506"
-					(reference "U$8")
+					(reference "J6")
 					(unit 1)
 				)
@@
 		(on_board yes)
 		(dnp no)
-		(property "Reference" "U$5"
+		(property "Reference" "J5"
 			(at 182.88 241.3 0)
 			(effects
@@
 			(project ""
 				(path "/f57eb5ac-0a1b-4ac0-915c-20e575439506"
-					(reference "U$5")
+					(reference "J5")
 					(unit 1)
 				)
@@
 		(on_board yes)
 		(dnp no)
-		(property "Reference" "U$100"
+		(property "Reference" "Y1"
 			(at 48.895 255.27 0)
 			(effects
@@
 			(project ""
 				(path "/f57eb5ac-0a1b-4ac0-915c-20e575439506"
-					(reference "U$100")
+					(reference "Y1")
 					(unit 1)
 				)
@@
 		(on_board yes)
 		(dnp no)
-		(property "Reference" "U$3"
+		(property "Reference" "J4"
 			(at 312.42 378.46 0)
 			(effects
@@
 			(project ""
 				(path "/f57eb5ac-0a1b-4ac0-915c-20e575439506"
-					(reference "U$3")
+					(reference "J4")
 					(unit 1)
 				)
@@
 		(on_board yes)
 		(dnp no)
-		(property "Reference" "U$1"
+		(property "Reference" "J1"
 			(at 495.3 91.44 0)
 			(effects
@@
 			(project ""
 				(path "/f57eb5ac-0a1b-4ac0-915c-20e575439506"
-					(reference "U$1")
+					(reference "J1")
 					(unit 1)
 				)
@@
 		(on_board yes)
 		(dnp no)
-		(property "Reference" "U$9"
+		(property "Reference" "J7"
 			(at 426.72 218.44 90)
 			(effects
@@
 			(project ""
 				(path "/f57eb5ac-0a1b-4ac0-915c-20e575439506"
-					(reference "U$9")
+					(reference "J7")
 					(unit 1)
 				)

Commit message: fix(sch): separate U5's RS-485 differential pair (Y+A / Z+B)
An EAGLE-import wiring defect had all four of U5 (ADM2587E)'s RS-485
pins -- Y, Z, A, B -- electrically bussed onto one node (via a stray
wire bridging the "RS485_P"-labeled bus to the "RS485_N"-labeled wire
at (430.53,278.13)-(430.53,279.4), plus B tapping directly into the
Y/A junction instead of the Z/N side). This shorted the two
differential-pair legs together -- the bus could not have worked.

Removed the stray P/N bridge wire and B's incorrect tap into the P-bus
junction; rewired B onto the existing Z/RS485_N wire run instead,
matching this repo's own documented design intent
(PCB/RS485-CANFD-TPM-upgrade.md SS2: "Y+A together onto RS485_P... Z+B
together onto RS485_N").

Verified via kicad-cli's authoritative netlist export (not the custom
analyzer, which had misread this net): /RS485_P now contains exactly
U5.10(Y), U5.13(A), J6.P$4, J7.P$4; /RS485_N now contains exactly
U5.11(Z), U5.12(B), J6.P$3, J7.P$3. ERC errors 19->18, including the
specific U5 pin_to_pin (Y/Z output conflict) violation resolving.

Co-Authored-By: Claude Sonnet 5 <noreply@anthropic.com>
Connections:
- net RS485_N: no longer J6.P$4, J7.P$4, U5.10 (Y), U5.13 (A)
- new net RS485_P: J6.P$4, J7.P$4, U5.10 (Y), U5.13 (A)
Changed lines of the file:
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@@
-	(wire
-		(pts
-			(xy 430.53 278.13) (xy 430.53 279.4)
-		)
-		(stroke
-			(width 0.1524)
-			(type solid)
-		)
-	)
 	(wire
 		(pts
@@
 	(wire
 		(pts
-			(xy 422.91 279.4) (xy 425.45 279.4)
-		)
-		(stroke
+			(xy 422.91 279.4) (xy 422.91 278.13)
+		)
+		(stroke
+			(width 0.1524)
+			(type solid)
+		)
+	)
+	(wire
+		(pts
+			(xy 422.91 278.13) (xy 430.53 278.13)
+		)
+		(stroke

Commit message: fix(sch): separate U6's CAN-FD logic pins onto their correct nets
An EAGLE-import defect had bussed 5 of U6 (ADM3055E)'s pins --
GND1, VCC, VIO, RXD, TXD -- onto one continuous wire trunk that
ultimately reached a +3V3 power symbol, silently shorting the chip's
logic ground, its 5V isoPower input, its 3.3V IO supply, and both its
CAN-FD RX/TX signal pins together. Each pin already had a correctly-
named local label sitting on that same over-merged wire (GND, +3V3,
CAN0_RX, CAN0_TX, +5V_ISO_CANFD) -- the labels were right, the
underlying wire topology was wrong, exactly the
"similar_label_and_power"/"multiple_net_names" class of EAGLE-import
defect this repo's TODO.md SS6 already catalogs.

Removed the 6 bridging wire segments and 7 now-invalid junction dots
that merged these into one node. VCC's dedicated "+5V_ISO_CANFD" label
would not attach validly to its wire under kicad-cli 9.0.2's ERC
regardless of placement tried (mid-wire, exact endpoint); removed it
rather than ship a label that doesn't do what it claims -- VCC is
still correctly reported as undriven by ERC (power_pin_not_driven /
pin_not_connected), matching this repo's own documented, deliberate
open item (PCB/RS485-CANFD-TPM-upgrade.md SS3: "VCC ... wired to a new
+5V_ISO_CANFD net that nothing currently drives ... deliberately left
as an open BOM/regulator-selection decision").

Verified via kicad-cli's authoritative netlist export: U6.1(GND1)->GND,
U6.3(VIO)->+3V3, U6.4(RXD)->/CAN0_RX (tied to U1.17, the MCU pin --
already correctly wired, just drowned out by the short), U6.6(TXD)->
/CAN0_TX (tied to U1.16), U6.5(SILENT)/U6.7(STBY)->GND, U6.2(VCC)->its
own isolated net. The fix also correctly re-isolated B5's ground leg
(previously shorted to +3V3) onto /CANFD_ISO_GND with GND2/RS, and
newly exposes U6's isolated-side pins (GND2/VISOIN/GNDISO/VISOOUT)
needing a PWR_FLAG -- the same treatment U5's analogous pins already
need, deferred to the ERC warning cleanup pass (TODO.md 6.2/6.3).

Co-Authored-By: C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
Connections:
- net +3V3: no longer #U$26.1 (P$1), #U$27.1 (P$1), B5.2, C1.1, C10.2, C11.2, C12.1, C13.1, C14.2, C15.2, C16.1, C17.1, C18.1, C19.1, C2.1, C20.2, C21.2, C22.-, C23.2, C24.2, C25.2, C26.2, C3.2, C31.1, C31.2, C32.1, C32.2, C33.2, C34.2, C37.2, C38.2, C39.2, C4.2, C40.2, C41.2, C42.2, C43.2, C44.2, C45.2, C46.2, C5.2, C6.2, C7.2, C8.1, C9.2, J3.P$2, J4.P$4, J5.P$3, J6.P$2, J7.P$2, M1.P$1 (G), M2.P$1 (S1_N), M3.P$1 (S1_N), M4.P$3 (GND), M4.P$9 (TP), M5.P$3 (GND), M5.P$9 (TP), NTC0.1, R11.2, R12.2, R20.2, R4.1, RV1.P$3, U1.16 (PA12/CAN0_TX), U1.17 (PA13/CAN0_RX), U1.25 (PA21/VREF-), U1.33 (PAD), U1.5 (VSS), U10.P$13, U10.P$20, U10.P$25, U2.P$12 (P$8_PGND), U2.P$13 (P$8_PGND), U2.P$14 (P$8_PGND), U3.2 (P$2), U4.P$10, U4.P$5, U4.P$7, U4.P$8, U4.P$9, U5.2 (GND1), U6.1 (GND1), U6.10 (RS), U6.2 (VCC), U6.4 (RXD), U6.5 (SILENT), U6.6 (TXD), U6.7 (STBY), U6.9 (GND2), U7.1 (GND), Y1.P$2 (GND)
- new net CAN0_RX: U1.17 (PA13/CAN0_RX), U6.4 (RXD)
- new net CAN0_TX: U1.16 (PA12/CAN0_TX), U6.6 (TXD)
- new net CANFD_ISO_GND: #U$26.1 (P$1), #U$27.1 (P$1), B5.2, C31.1, C32.1, C37.2, C38.2, C41.2, U6.10 (RS), U6.9 (GND2)
- new net GND: C1.1, C10.2, C11.2, C12.1, C13.1, C14.2, C15.2, C16.1, C17.1, C18.1, C19.1, C2.1, C20.2, C21.2, C22.-, C23.2, C24.2, C25.2, C26.2, C3.2, C31.2, C32.2, C33.2, C34.2, C39.2, C4.2, C40.2, C42.2, C43.2, C44.2, C45.2, C46.2, C5.2, C6.2, C7.2, C8.1, C9.2, J3.P$2, J4.P$4, J5.P$3, J6.P$2, J7.P$2, M1.P$1 (G), M2.P$1 (S1_N), M3.P$1 (S1_N), M4.P$3 (GND), M4.P$9 (TP), M5.P$3 (GND), M5.P$9 (TP), NTC0.1, R11.2, R12.2, R20.2, R4.1, RV1.P$3, U1.25 (PA21/VREF-), U1.33 (PAD), U1.5 (VSS), U10.P$13, U10.P$20, U10.P$25, U2.P$12 (P$8_PGND), U2.P$13 (P$8_PGND), U2.P$14 (P$8_PGND), U3.2 (P$2), U4.P$10, U4.P$5, U4.P$7, U4.P$8, U4.P$9, U5.2 (GND1), U6.1 (GND1), U6.5 (SILENT), U6.7 (STBY), U7.1 (GND), Y1.P$2 (GND)
Changed lines of the file:
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@@
 	)
 	(junction
-		(at 68.58 392.43)
-		(diameter 0)
-		(color 0 0 0 0)
-	)
-	(junction
 		(at 406.4 119.38)
 		(diameter 0)
@@
 	)
 	(junction
-		(at 68.58 387.35)
-		(diameter 0)
-		(color 0 0 0 0)
-	)
-	(junction
 		(at 416.56 114.3)
 		(diameter 0)
@@
 	)
 	(junction
-		(at 63.5 400.05)
-		(diameter 0)
-		(color 0 0 0 0)
-	)
-	(junction
 		(at 416.56 96.52)
 		(diameter 0)
@@
 	)
 	(junction
-		(at 63.5 392.43)
-		(diameter 0)
-		(color 0 0 0 0)
-	)
-	(junction
 		(at 431.8 269.24)
 		(diameter 0)
@@
 	)
 	(junction
-		(at 63.5 389.89)
-		(diameter 0)
-		(color 0 0 0 0)
-	)
-	(junction
 		(at 73.66 248.92)
 		(diameter 0)
@@
 	)
 	(junction
-		(at 63.5 394.97)
-		(diameter 0)
-		(color 0 0 0 0)
-	)
-	(junction
 		(at 406.4 71.12)
 		(diameter 0)
@@
 	)
 	(junction
-		(at 63.5 387.35)
-		(diameter 0)
-		(color 0 0 0 0)
-	)
-	(junction
 		(at 147.32 304.8)
 		(diameter 0)
@@
 	(wire
 		(pts
-			(xy 68.58 387.35) (xy 68.58 392.43)
-		)
-		(stroke
-			(width 0.1524)
-			(type solid)
-		)
-	)
-	(wire
-		(pts
 			(xy 63.5 369.57) (xy 58.42 369.57)
 		)
@@
 		)
 	)
-	(wire
-		(pts
-			(xy 63.5 392.43) (xy 63.5 394.97)
-		)
-		(stroke
-			(width 0.1524)
-			(type solid)
-		)
-	)
 	(polyline
 		(pts
@@
 	(wire
 		(pts
-			(xy 63.5 400.05) (xy 63.5 415.29)
-		)
-		(stroke
-			(width 0.1524)
-			(type solid)
-		)
-	)
-	(wire
-		(pts
 			(xy 130.48 402.59) (xy 130.48 435.61)
 		)
@@
 	(wire
 		(pts
-			(xy 63.5 400.05) (xy 63.5 394.97)
-		)
-		(stroke
-			(width 0.1524)
-			(type solid)
-		)
-	)
-	(wire
-		(pts
 			(xy 464.82 134.62) (xy 490.22 134.62)
 		)
@@
 	(wire
 		(pts
-			(xy 63.5 389.89) (xy 63.5 387.35)
-		)
-		(stroke
-			(width 0.1524)
-			(type solid)
-		)
-	)
-	(wire
-		(pts
 			(xy 368.3 193.04) (xy 365.76 193.04)
 		)
@@
 	(wire
 		(pts
-			(xy 63.5 389.89) (xy 63.5 392.43)
-		)
-		(stroke
-			(width 0.1524)
-			(type solid)
-		)
-	)
-	(wire
-		(pts
 			(xy 203.2 238.76) (xy 203.2 236.22)
 		)
@@
 		)
 	)
-	(label "+5V_ISO_CANFD"
-		(at 63.5 415.29 0)
-		(effects
-			(font
-				(size 1.1735 1.1735)
-			)
-			(justify left bottom)
-		)
-	)
